File: kicad/_autosave-Trackball.kicad_pcb (KiCad board)
At the start: 2 copper layers, 60 x 55 mm, 31 parts, among them J1 Conn_01x04, J101 Conn_02x03_Counter_Clockwise, SW1 Push_Button, SW102 Push_Button, SW103 Push_Button, SW106 Push_Button, SW2 Push_Button, SW3 RotaryEncoder_Switch_MP, U103 TCR2EF19, U2 PMW3360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

Commit message: up
Routing:
- net EN: track 41.8 -> 37.3 mm
- net +3V3: track 100.0 -> 101.6 mm
- net Net-(SW102-B): track 11.9 -> 12.4 mm
- net GND: vias 22 -> 674
