File: V02/MaSe/MaSe.kicad_pcb (KiCad board)
At the start: 2 copper layers, 63.8 x 97.6 mm, 44 parts, among them J1 Conn_02x08_Odd_Even, J2 ALIM_BAT, J3 Conn_02x08_Odd_Even, J4 Conn_01x02, Q2 BSS83P, Q3 BSS83P, SW1 Push_Button, SW10 Push_Button, SW2 Push_Button, SW3 RotaryEncoder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

Commit message: fist POC
Routing:
- net +3V3: track 145.1 -> 145.7 mm
